Commit message: replase the small blocks of maze with bigger ones

File: Husky+Arm(puru2411)/cubes/urdf/10y_segment.urdf (robot description, URDF)
Before this commit: robot cube.urdf, 2 links, 1 joints
Links:
- link baseLink: geometry collision box size=.1 10 .4; visual mesh filename=cubes/meshes/cube.obj scale=.1 10 .4

File: Husky+Arm(puru2411)/cubes/urdf/4x_segment.urdf (robot description, URDF)
Before this commit: robot cube.urdf, 2 links, 1 joints
Links:
- link baseLink: geometry collision box size=4 .1 .4; visual mesh filename=cubes/meshes/cube.obj scale=4 .1 .4

File: Husky+Arm(puru2411)/cubes/urdf/6y_segment.urdf (robot description, URDF)
Before this commit: robot cube.urdf, 2 links, 1 joints
Links:
- link baseLink: geometry collision box size=.1 6 .4; visual mesh filename=cubes/meshes/cube.obj scale=.1 6 .4
